File: schematic/schematic.kicad_sch (KiCad schematic)
At the start: 32 parts, among them J1 Conn_01x03_Socket, J2 Conn_01x03_Socket, Q1 BC327, Q2 BC327, Q3 BC327, Q4 BC327, U1 ATmega328-P, U2 5161BS, U3 5161BS, U4 5161BS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

Commit message: added file viewer
Parts:
- C4: value 1000uF -> 250uF
Other:
- moved on the sheet: R3
Changed lines of the file:
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@@
 	(wire
 		(pts
-			(xy 139.7 33.02) (xy 138.43 33.02)
-		)
-		(stroke
-			(width 0)
-			(type default)
-		)
-	)
-	(wire
-		(pts
 			(xy 219.71 72.39) (xy 219.71 73.66)
 		)
@@
 		)
 	)
-	(label "Tester"
-		(at 247.65 116.84 0)
-		(effects
-			(font
-				(size 1.27 1.27)
-			)
-			(justify left bottom)
-		)
-	)
 	(global_label "SEGE"
 		(shape input)
@@
 	(global_label "D3"
 		(shape input)
-		(at 138.43 27.94 90)
+		(at 139.7 27.94 90)
 		(fields_autoplaced yes)
 		(effects
@@
 		)
 		(property "Intersheetrefs" "${INTERSHEET_REFS}"
-			(at 138.43 22.4753 90)
+			(at 139.7 22.4753 90)
 			(hide yes)
 			(show_name no)
@@
 		)
 	)
+	(global_label "Tester"
+		(shape input)
+		(at 247.65 116.84 180)
+		(fields_autoplaced yes)
+		(effects
+			(font
+				(size 1.27 1.27)
+			)
+			(justify right)
+		)
+		(property "Intersheetrefs" "${INTERSHEET_REFS}"
+			(at 238.98 116.84 0)
+			(hide yes)
+			(show_name no)
+			(do_not_autoplace no)
+			(effects
+				(font
+					(size 1.27 1.27)
+				)
+				(justify right)
+			)
+		)
+	)
 	(global_label "SEGA_CTRL"
 		(shape input)
@@
 	(symbol
 		(lib_id "Device:R_Small_US")
-		(at 138.43 30.48 0)
+		(at 139.7 30.48 0)
 		(mirror y)
 		(unit 1)
@@
 		(fields_autoplaced yes)
 		(property "Reference" "R3"
-			(at 135.89 29.2099 0)
+			(at 137.16 29.2099 0)
 			(show_name no)
 			(do_not_autoplace no)
@@
 		)
 		(property "Value" "4.7k"
-			(at 135.89 31.7499 0)
+			(at 137.16 31.7499 0)
 			(show_name no)
 			(do_not_autoplace no)
@@
 		)
 		(property "Footprint" ""
-			(at 138.43 30.48 0)
+			(at 139.7 30.48 0)
 			(hide yes)
 			(show_name no)
@@
 		)
 		(property "Datasheet" ""
-			(at 138.43 30.48 0)
+			(at 139.7 30.48 0)
 			(hide yes)
 			(show_name no)
@@
 		)
 		(property "Description" "Resistor, small US symbol"
-			(at 138.43 30.48 0)
+			(at 139.7 30.48 0)
 			(hide yes)
 			(show_name no)
@@
 			)
 		)
-		(property "Value" "1000uF"
+		(property "Value" "250uF"
 			(at 257.81 38.1062 0)
 			(show_name no)
